File: HW/ledpwmble/DEBUG.sch (KiCad schematic (older format))
At the start: 5 parts

Commit message: HW: Rev 1 - 1922
Parts:
- C21: footprint Capacitors_SMD:C_0805_HandSoldering -> Capacitor_SMD:C_0603_1608Metric
- CON1: renamed from CON?; footprint (none) -> athir:HFW6R_2STE1LF
- R19, R20, R21: footprint Resistors_SMD:R_0805_HandSoldering -> Resistor_SMD:R_0603_1608Metric
Connections:
- no-connect marks 0 -> 1
Changed lines of the file:
@@
 F 0 "R19" H 3180 3145 50  0000 L CNN
 F 1 "100kohm" V 3200 3225 50  0000 L CNN
-F 2 "Resistors_SMD:R_0805_HandSoldering" H 3150 3125 50  0001 C CNN
+F 2 "Resistor_SMD:R_0603_1608Metric" H 3150 3125 50  0001 C CNN
 F 3 "" H 3150 3125 50  0000 C CNN
 	1    3150 3125
@@
 F 0 "R20" H 3380 2945 50  0000 L CNN
 F 1 "100kohm" V 3400 3025 50  0000 L CNN
-F 2 "Resistors_SMD:R_0805_HandSoldering" H 3350 2925 50  0001 C CNN
+F 2 "Resistor_SMD:R_0603_1608Metric" H 3350 2925 50  0001 C CNN
 F 3 "" H 3350 2925 50  0000 C CNN
 	1    3350 2925
@@
 F 0 "R21" H 3580 3145 50  0000 L CNN
 F 1 "100kohm" V 3600 3225 50  0000 L CNN
-F 2 "Resistors_SMD:R_0805_HandSoldering" H 3550 3125 50  0001 C CNN
+F 2 "Resistor_SMD:R_0603_1608Metric" H 3550 3125 50  0001 C CNN
 F 3 "" H 3550 3125 50  0000 C CNN
 	1    3550 3125
@@
 F 0 "C21" H 3260 3920 50  0000 L CNN
 F 1 "100nF" H 3260 3770 50  0000 L CNN
-F 2 "Capacitors_SMD:C_0805_HandSoldering" H 3250 3850 50  0001 C CNN
+F 2 "Capacitor_SMD:C_0603_1608Metric" H 3250 3850 50  0001 C CNN
 F 3 "" H 3250 3850 50  0000 C CNN
 	1    3250 3850
@@
 	3550 3400 2900 3400
 $Comp
-L fpc_conn:FPC_6POS CON?
+L fpc_conn:FPC_6POS CON1
 U 1 1 5CF30BC9
 P 4200 3800
-F 0 "CON?" H 4278 4045 60  0000 L CNN
+F 0 "CON1" H 4278 4045 60  0000 L CNN
 F 1 "FPC_6POS" H 4278 3939 60  0000 L CNN
-F 2 "" H 4200 3800 60  0001 C CNN
+F 2 "athir:HFW6R_2STE1LF" H 4200 3800 60  0001 C CNN
 F 3 "" H 4200 3800 60  0001 C CNN
 	1    4200 3800
@@
 	2900 3700 3750 3700
 $Comp
-L power:GND #PWR?
+L power:GND #PWR0116
 U 1 1 5CF340D9
 P 3700 4025
-F 0 "#PWR?" H 3700 3775 50  0001 C CNN
+F 0 "#PWR0116" H 3700 3775 50  0001 C CNN
 F 1 "GND" H 3705 3852 50  0000 C CNN
 F 2 "" H 3700 4025 50  0001 C CNN
@@
 Wire Wire Line
 	3700 3800 3750 3800
+NoConn ~ 4100 4100
 $EndSCHEMATC

Commit message: Sorry?
Changed lines of the file:
@@
 L power:GND #PWR043
 U 1 1 58891062
-P 3250 4025
-F 0 "#PWR043" H 3250 3775 50  0001 C CNN
-F 1 "GND" H 3250 3875 50  0000 C CNN
-F 2 "" H 3250 4025 50  0000 C CNN
-F 3 "" H 3250 4025 50  0000 C CNN
-	1    3250 4025
+P 3250 4000
+F 0 "#PWR043" H 3250 3750 50  0001 C CNN
+F 1 "GND" H 3250 3850 50  0000 C CNN
+F 2 "" H 3250 4000 50  0000 C CNN
+F 3 "" H 3250 4000 50  0000 C CNN
+	1    3250 4000
 	1    0    0    -1
 $EndComp
-Wire Wire Line
-	3250 4025 3250 3950
 Wire Wire Line
 	3550 3225 3550 3400
@@
 	3700 3800 3750 3800
 NoConn ~ 4100 4100
+Wire Wire Line
+	3250 3950 3250 4000
 $EndSCHEMATC
