File: HW/ledpwmble/ledpwmble.kicad_pcb (KiCad board)
At the start: 2 copper layers, 55.6 x 30 mm, 39 parts, among them CON1 FPC_6POS, IC1 ATSAMD21G18A-AU, J1 Conn_01x08, Q1 NTR5103NT1G, Q2 NTR5103NT1G, Q3 NTR5103NT1G, U1 MIC5504-3.3YM5, U2 TPS62173DSG, Y1 Crystal_Small

Commit message: Sorry?
Connections:
- C3 pad 2: Net-(C3-Pad2) -> GND
- C4 pad 2: Net-(C3-Pad2) -> GND
- U1 pad 2: Net-(C3-Pad2) -> GND
Routing:
- net GND: track 10.5 -> 22.1 mm, vias 60 -> 62
- net Net-(C3-Pad2): track 11.6 -> 0.00 mm, vias 2 -> 0
