File: HW/ledpwmble/ledpwmble.sch (KiCad schematic (older format))
At the start: 27 parts

Commit message: HW: Rev 1 - 1922
Parts:
- C1, C2, C3, C4, C5, C6, C7, C8: renamed from C?; footprint (none) -> Capacitor_SMD:C_0603_1608Metric
- D1, D2, D3: renamed from D?; footprint (none) -> TestPoint:TestPoint_2Pads_Pitch2.54mm_Drill0.8mm
- FL1: renamed from FL?; footprint (none) -> athir:ACP3225
- IC1: renamed from IC?; footprint QFP50P900X900X120-48N -> Package_QFP:TQFP-48_7x7mm_P0.5mm
- J1: renamed from J?; footprint (none) -> Connector_PinSocket_2.54mm:PinSocket_1x08_P2.54mm_Vertical
- L2: renamed from L?; footprint (none) -> Inductor_SMD:L_Wuerth_MAPI-3020
- Q1, Q2, Q3: renamed from Q?; footprint TO_SOT_Packages_THT:TO-220_Vertical -> Package_TO_SOT_SMD:SOT-23
- R1, R2, R3, R4: renamed from R?; footprint (none) -> Resistor_SMD:R_0603_1608Metric
- TP1, TP2: renamed from TP?; footprint (none) -> TestPoint:TestPoint_Plated_Hole_D3.0mm
- Y1: renamed from Y?; footprint (none) -> Crystal:Crystal_SMD_3215-2Pin_3.2x1.5mm
- gave numbers to parts that had none: 2
Connections:
- net +5V: no longer C7.2, C8.2, U2.5 (FB)
- new net: C7.2, C8.2, U2.5 (FB)

Commit message: Sorry?
Connections:
- net GND: now also C3.2, C4.2, U1.2 (GND)
- no-connect marks 3 -> 31
Other:
- moved on the sheet: C4
Changed lines of the file:
@@
 L power:GND #PWR0103
 U 1 1 5CF41704
-P 2925 4300
-F 0 "#PWR0103" H 2925 4050 50  0001 C CNN
-F 1 "GND" H 2930 4127 50  0000 C CNN
-F 2 "" H 2925 4300 50  0001 C CNN
-F 3 "" H 2925 4300 50  0001 C CNN
-	1    2925 4300
+P 2925 4325
+F 0 "#PWR0103" H 2925 4075 50  0001 C CNN
+F 1 "GND" H 2930 4152 50  0000 C CNN
+F 2 "" H 2925 4325 50  0001 C CNN
+F 3 "" H 2925 4325 50  0001 C CNN
+	1    2925 4325
 	1    0    0    -1
 $EndComp
@@
 Wire Wire Line
 	3025 4275 2925 4275
-Wire Wire Line
-	2925 4275 2925 4300
 Wire Wire Line
 	2925 4275 2850 4275
@@
 Wire Wire Line
 	3600 1675 3600 1875
-Wire Wire Line
-	3600 1875 4275 1875
-Wire Wire Line
-	4275 1875 4275 1825
 $Comp
 L Device:CP_Small C4
 U 1 1 5CFCCF95
-P 4825 1550
-F 0 "C4" H 4913 1596 50  0000 L CNN
-F 1 "10uF" H 4913 1505 50  0000 L CNN
-F 2 "Capacitor_SMD:C_0603_1608Metric" H 4825 1550 50  0001 C CNN
-F 3 "~" H 4825 1550 50  0001 C CNN
-	1    4825 1550
-	1    0    0    -1
-$EndComp
-Wire Wire Line
-	4825 1450 4825 1425
+P 4825 1625
+F 0 "C4" H 4913 1671 50  0000 L CNN
+F 1 "10uF" H 4913 1580 50  0000 L CNN
+F 2 "Capacitor_SMD:C_0603_1608Metric" H 4825 1625 50  0001 C CNN
+F 3 "~" H 4825 1625 50  0001 C CNN
+	1    4825 1625
+	1    0    0    -1
+$EndComp
+Wire Wire Line
+	4825 1525 4825 1425
 Wire Wire Line
 	4825 1425 4675 1425
 Wire Wire Line
-	4825 1650 4825 1875
-Wire Wire Line
-	4825 1875 4275 1875
-Connection ~ 4275 1875
+	4825 1725 4825 1875
 $Comp
 L power:VCC #PWR0115
@@
 F 3 "" H 10225 1175 50  0001 C CNN
 	1    10225 1175
-	1    0    0    -1
-$EndComp
-$Comp
-L power:VCC #PWR0119
-U 1 1 5CF48ADC
-P 10400 1175
-F 0 "#PWR0119" H 10400 1025 50  0001 C CNN
-F 1 "VCC" H 10417 1348 50  0000 C CNN
-F 2 "" H 10400 1175 50  0001 C CNN
-F 3 "" H 10400 1175 50  0001 C CNN
-	1    10400 1175
 	1    0    0    -1
 $EndComp
@@
 Wire Wire Line
 	10225 1275 10225 1175
+Wire Wire Line
+	3600 1875 4275 1875
+Wire Wire Line
+	4275 1825 4275 1875
+Connection ~ 4275 1875
+Wire Wire Line
+	4275 1875 4825 1875
+$Comp
+L power:GND #PWR0120
+U 1 1 5CFEEF53
+P 4275 2000
+F 0 "#PWR0120" H 4275 1750 50  0001 C CNN
+F 1 "GND" H 4280 1827 50  0000 C CNN
+F 2 "" H 4275 2000 50  0001 C CNN
+F 3 "" H 4275 2000 50  0001 C CNN
+	1    4275 2000
+	1    0    0    -1
+$EndComp
+Wire Wire Line
+	4275 2000 4275 1875
+NoConn ~ 4500 3875
+NoConn ~ 4500 3975
+NoConn ~ 4500 4075
+NoConn ~ 4500 4175
+NoConn ~ 4500 4375
+NoConn ~ 4500 4475
+NoConn ~ 3300 3975
+NoConn ~ 3300 4075
+NoConn ~ 3300 4175
+NoConn ~ 3300 4275
+NoConn ~ 3300 4375
+NoConn ~ 3300 4475
+NoConn ~ 3300 4675
+NoConn ~ 3300 4875
+NoConn ~ 3300 5075
+NoConn ~ 3300 5275
+NoConn ~ 3300 5375
+NoConn ~ 3300 5475
+NoConn ~ 3300 5575
+NoConn ~ 3300 5675
+NoConn ~ 3300 5775
+NoConn ~ 3300 5875
+NoConn ~ 3300 5975
+NoConn ~ 3300 6075
+NoConn ~ 3300 6175
+NoConn ~ 3300 6275
+NoConn ~ 3300 6375
+NoConn ~ 3300 6475
+Wire Wire Line
+	2925 4275 2925 4325
 $Comp
 L power:PWR_FLAG #FLG0103
-U 1 1 5CF5319F
-P 10400 1275
-F 0 "#FLG0103" H 10400 1350 50  0001 C CNN
-F 1 "PWR_FLAG" H 10400 1448 50  0000 C CNN
-F 2 "" H 10400 1275 50  0001 C CNN
-F 3 "~" H 10400 1275 50  0001 C CNN
-	1    10400 1275
+U 1 1 5D06E2E2
+P 10500 1275
+F 0 "#FLG0103" H 10500 1350 50  0001 C CNN
+F 1 "PWR_FLAG" H 10500 1448 50  0000 C CNN
+F 2 "" H 10500 1275 50  0001 C CNN
+F 3 "~" H 10500 1275 50  0001 C CNN
+	1    10500 1275
 	-1   0    0    1
 $EndComp
-Wire Wire Line
-	10400 1275 10400 1175
+$Comp
+L power:GND #PWR0119
+U 1 1 5D06E71F
+P 10725 1275
+F 0 "#PWR0119" H 10725 1025 50  0001 C CNN
+F 1 "GND" H 10730 1102 50  0000 C CNN
+F 2 "" H 10725 1275 50  0001 C CNN
+F 3 "" H 10725 1275 50  0001 C CNN
+	1    10725 1275
+	1    0    0    -1
+$EndComp
+Wire Wire Line
+	10725 1275 10725 1200
+Wire Wire Line
+	10725 1200 10500 1200
+Wire Wire Line
+	10500 1200 10500 1275
 $EndSCHEMATC
